File: picamera-hdmi.sch (KiCad schematic (older format))
At the start: 4 parts, among them J1 FPC68611514122, J2 HDMI-685119136923, J3 Conn_01x05, J4 Conn_01x02

Commit message: more info in schematic
Parts:
- J2: digikey-part (none) -> 732-2739-1-ND
Connections:
- no-connect marks 2 -> 1
Other:
- note added: "<— FFC to Pi Camera / to Raspberry Pi"
- note added: "HDMI cable —>"
- note added: "L. Riegger 2018"
- note added: "breakout supply voltage"
- note added: "breakout unused HDMI pins"
- note added: "picamera-hdmi"
- note added: "picamera-hdmi\nconverter from Pi Camera FFC to (mini) HDMI"
- note added: "v1.0"
- moved on the sheet: J1, J2, J3, J4
